Commit message: Added irb120_support to rtbdata

File: rtb-data/rtbdata/xacro/abb_irb140/urdf/irb140.urdf (robot description, URDF)
Before this commit: robot abb_irb140, 9 links, 8 joints
Links:
- link base_link: geometry collision mesh filename=package://abb_irb140/meshes/irb140/collision/base_link.stl; visual mesh filename=package://abb_irb140/meshes/irb140/visual/base_link.stl
- link link_1: geometry collision mesh filename=package://abb_irb140/meshes/irb140/collision/link_1.stl; visual mesh filename=package://abb_irb140/meshes/irb140/visual/link_1.stl
- link link_2: geometry collision mesh filename=package://abb_irb140/meshes/irb140/collision/link_2.stl; visual mesh filename=package://abb_irb140/meshes/irb140/visual/link_2.stl
- link link_3: geometry collision mesh filename=package://abb_irb140/meshes/irb140/collision/link_3.stl; visual mesh filename=package://abb_irb140/meshes/irb140/visual/link_3.stl
- link link_4: geometry collision mesh filename=package://abb_irb140/meshes/irb140/collision/link_4.stl; visual mesh filename=package://abb_irb140/meshes/irb140/visual/link_4.stl
- link link_5: geometry collision mesh filename=package://abb_irb140/meshes/irb140/collision/link_5.stl; visual mesh filename=package://abb_irb140/meshes/irb140/visual/link_5.stl
- link link_6: geometry collision mesh filename=package://abb_irb140/meshes/irb140/collision/link_6.stl; visual mesh filename=package://abb_irb140/meshes/irb140/visual/link_6.stl
